File: Feeder.sch (KiCad schematic (older format))
At the start: 13 parts, among them J1 UPDI, J2 Internal, J3 RS485, Q1 2N7002NXAKR, U1 ATtiny402, U2 ST485EBDR

Commit message: Fix ATTiny402-SS part reference
Parts:
- U1: symbol Feeder-rescue:ATtiny402-SS-MCU_Microchip_ATtiny -> MCU_Microchip_ATtiny:ATtiny402-SS
Changed lines of the file:
@@
 $EndDescr
 $Comp
-L Feeder-rescue:ATtiny402-SS-MCU_Microchip_ATtiny U1
+L MCU_Microchip_ATtiny:ATtiny402-SS U1
 U 1 1 5E2EEF2E
 P 3400 1650

Commit message: Invert Motor and Feedback: Allow to use UPDI pin always as input and may avoid damaged IC
Parts:
- added R3: 1k, Resistor_SMD:R_0402_1005Metric, symbol Device:R_Small
Connections:
- net labels added: MOTOR
- net labels removed: UPDI
- wire segments 74 -> 75
Changed lines of the file:
@@
 Sheet 1 1
 Title "PNP Feeder"
-Date "2020-03-30"
+Date "2021-05-29"
 Rev ""
 Comp ""
@@
 $EndComp
 Wire Wire Line
-	4000 1350 4625 1350
-Text Label 4625 1350 0    50   ~ 0
-UPDI
+	4000 1350 4825 1350
+Text Label 4825 1550 2    50   ~ 0
+MOTOR
 Wire Wire Line
 	1575 2950 1525 2950
 Text Label 1525 3050 2    50   ~ 0
-UPDI
+FEEDBACK
 Wire Wire Line
 	6025 1850 6125 1850
@@
 Wire Wire Line
 	4250 4750 4975 4750
-Text Label 4400 4950 0    50   ~ 0
+Text Label 4700 4950 0    50   ~ 0
 FEEDBACK
 Wire Wire Line
 	5100 1450 5100 1750
-Text Label 4825 1550 2    50   ~ 0
+Text Label 4825 1350 2    50   ~ 0
 FEEDBACK
 Wire Wire Line
@@
 F 1 "2N7002NXAKR" H 4550 4675 50  0000 L CNN
 F 2 "Package_TO_SOT_SMD:SOT-23" H 5275 4625 50  0001 C CNN
-F 3 "~" H 5075 4525 50  0001 C CNN
+F 3 "https://assets.nexperia.com/documents/data-sheet/2N7002NXAK.pdf" H 5075 4525 50  0001 C CNN
 	1    5075 4525
 	-1   0    0    -1
@@
 	5325 4525 5325 4550
 Text Label 5600 4525 2    50   ~ 0
-UPDI
+MOTOR
 Wire Wire Line
 	5600 4525 5325 4525
@@
 Wire Wire Line
 	4500 4850 4500 4600
+$Comp
+L Device:R_Small R3
+U 1 1 60B20362
+P 4500 4950
+F 0 "R3" H 4559 4996 50  0000 L CNN
+F 1 "1k" H 4559 4905 50  0000 L CNN
+F 2 "Resistor_SMD:R_0402_1005Metric" H 4500 4950 50  0001 C CNN
+F 3 "~" H 4500 4950 50  0001 C CNN
+	1    4500 4950
+	0    1    1    0
+$EndComp
+Wire Wire Line
+	4600 4950 4700 4950
 $EndSCHEMATC
